Commit message: Fix for HoloOcean COM offset

File: coug_ws/src/coug_description/urdf/bluerov2_holoocean/bluerov2_holoocean.urdf.xacro (robot description, xacro)
@@ -11,13 +11,6 @@
   <xacro:property name="iyy" value="0.17" />
   <xacro:property name="izz" value="0.12" />
-  <!-- Fix for matching CougUV URDF -->
-  <link name="base_link"/>
-  <joint name="com_joint" type="fixed">
-    <parent link="base_link"/>
-    <child link="com_link"/>
-    <origin xyz="0 0 0" rpy="0 0 0"/>
-  </joint>
   <!-- Main BlueROV2 body -->
-  <link name="com_link">
+  <link name="base_link">
     <visual>
       <geometry>
@@ -27,4 +20,11 @@
   </link>
   <!-- NOTE: These are exact HoloOcean socket locations as of 2.0.1 -->
+  <!-- COM -->
+  <joint name="com_joint" type="fixed">
+    <parent link="base_link"/>
+    <child link="com_link"/>
+    <origin xyz="0 0 0" rpy="0 0 0"/>
+  </joint>
+  <link name="com_link"/>
   <!-- IMUSocket -->
   <joint name="imu_joint" type="fixed">

File: coug_ws/src/coug_description/urdf/couguv_holoocean.urdf.xacro (robot description, xacro)
@@ -32,5 +32,5 @@
   <!-- Function to generate fins -->
   <xacro:macro name="fin_macro" params="prefix rpy_str">
-    <joint name="${prefix}_fin_joint" type="revolute"> <parent link="com_link"/>
+    <joint name="${prefix}_fin_joint" type="revolute"> <parent link="base_link"/>
       <child link="${prefix}_fin_link"/>
       <origin xyz="${-fin_offset} 0 0" rpy="${rpy_str}"/>
@@ -48,13 +48,6 @@
       </link>
   </xacro:macro>
-  <!-- Account for HoloOcean COM offset -->
-  <link name="base_link"/>
-  <joint name="com_joint" type="fixed">
-    <parent link="base_link"/>
-    <child link="com_link"/>
-    <origin xyz="0.1 0 0.1" rpy="0 0 0"/>
-  </joint>
   <!-- Main AUV body -->
-  <link name="com_link">
+  <link name="base_link">
     <visual>
       <origin xyz="0 0 0" rpy="0 ${pi/2} 0"/>
@@ -67,5 +60,5 @@
   <!-- Handle -->
   <joint name="handle_joint" type="fixed">
-    <parent link="com_link"/>
+    <parent link="base_link"/>
     <child link="handle_link"/>
     <origin xyz="0 0 ${base_radius}" rpy="0 0 0"/>
@@ -82,5 +75,5 @@
   <!-- Weight tray -->
   <joint name="tray_joint" type="fixed">
-    <parent link="com_link"/>
+    <parent link="base_link"/>
     <child link="tray_link"/>
     <origin xyz="0 0 -${base_radius}" rpy="0 0 0"/>
@@ -97,5 +90,5 @@
   <!-- Front hull -->
   <joint name="hull_joint" type="fixed">
-    <parent link="com_link"/>
+    <parent link="base_link"/>
     <child link="hull_link"/>
     <origin xyz="${(base_length-2*base_radius)/2} 0 0" rpy="0 0 0"/>
@@ -112,5 +105,5 @@
   <!-- Thruster -->
   <joint name="thruster_joint" type="fixed">
-    <parent link="com_link"/>
+    <parent link="base_link"/>
     <child link="thruster_link"/>
      <origin xyz="${-(base_length-2*base_radius)/2} 0 0" rpy="0 0 0"/>
@@ -130,4 +123,11 @@
   <xacro:fin_macro prefix="right" rpy_str="${-pi*2/3} 0 0"/>
   <!-- NOTE: These are exact HoloOcean socket locations as of 2.0.1 -->
+  <!-- COM -->
+  <joint name="com_joint" type="fixed">
+    <parent link="base_link"/>
+    <child link="com_link"/>
+    <origin xyz="0.0 0 0.0" rpy="0 0 0"/>
+  </joint>
+  <link name="com_link"/>
   <!-- IMUSocket -->
   <joint name="imu_joint" type="fixed">
